Commit message: Update rover_full.urdf.xacro

File: rover_description/urdf/rover_full.urdf.xacro (robot description, xacro)
@@ -1 +1,35 @@
-<?xml version="1.0"?><robot name="six_wheel_rover"><link name="base_link"/></robot>
+<?xml version="1.0"?>
+<robot name="six_wheel_rover" xmlns:xacro="http://ros.org/wiki/xacro">
+  <xacro:property name="wheel_radius" value="0.08"/>
+  <link name="base_link">
+    <inertial>
+      <mass value="25.0"/>
+      <origin xyz="0 0 0"/>
+      <inertia ixx="1.0" ixy="0.0" ixz="0.0" iyy="1.0" iyz="0.0" izz="1.0"/>
+    </inertial>
+  </link>
+  <!-- Front-left steering -->
+  <link name="fl_steer_link"/>
+  <joint name="fl_steer_joint" type="continuous">
+    <parent link="base_link"/>
+    <child link="fl_steer_link"/>
+    <origin xyz="0.35 0.25 0.0" rpy="0 0 0"/>
+    <axis xyz="0 0 1"/>
+  </joint>
+  <!-- Front-left wheel -->
+  <link name="fl_wheel_link"/>
+  <joint name="fl_wheel_joint" type="continuous">
+    <parent link="fl_steer_link"/>
+    <child link="fl_wheel_link"/>
+    <origin xyz="0 0 -0.08" rpy="0 0 0"/>
+    <axis xyz="0 1 0"/>
+  </joint>
+  <!-- Arm base (front center) -->
+  <link name="arm_base_link"/>
+  <joint name="arm_base_joint" type="fixed">
+    <parent link="base_link"/>
+    <child link="arm_base_link"/>
+    <origin xyz="0.45 0 0.2"/>
+  </joint>
+  <!-- Add rest of wheels, steers and arm joints similarly -->
+</robot>

Commit message: Update rover_full.urdf.xacro

File: rover_description/urdf/rover_full.urdf.xacro (robot description, xacro)
@@ -1,35 +1,420 @@
 <?xml version="1.0"?>
-<robot name="six_wheel_rover" xmlns:xacro="http://ros.org/wiki/xacro">
-  <xacro:property name="wheel_radius" value="0.08"/>
-  <link name="base_link">
+<!-- rover_full.urdf.xacro
+     Six-wheeled rover: 6 wheels (FL, ML, RL on left and FR, MR, RR on right)
+     Four steering joints: FL, FR, RL, RR (corner servos)
+     5-DOF arm mounted at front center
+     - All key dimensions are parameters at the top for easy tuning.
+     - Includes transmissions suitable for ros_control (velocity for wheels, position for steering, position/trajectory for arm).
+     - Basic Gazebo plugin placeholders for imu, kinect (rgbd), and gps.
+-->
+<robot xmlns:xacro="http://www.ros.org/wiki/xacro" name="six_wheel_rover">
+  <!-- ============================
+       USER-TUNABLE PARAMETERS
+       Edit these values to match your hardware
+       ============================ -->
+  <xacro:property name="wheel_radius" value="0.08"/>        <!-- meters -->
+  <xacro:property name="wheel_thickness" value="0.04"/>
+  <xacro:property name="track" value="0.7"/>               <!-- distance between left & right -->
+  <xacro:property name="half_track" value="${track/2.0}"/>
+  <xacro:property name="front_axle_x" value="0.45"/>
+  <xacro:property name="mid_axle_x" value="0.0"/>
+  <xacro:property name="rear_axle_x" value="-0.45"/>
+  <xacro:property name="base_length" value="0.9"/>
+  <xacro:property name="base_width" value="${track}"/>
+  <xacro:property name="base_height" value="0.18"/>
+  <xacro:property name="wheel_mass" value="0.8"/>
+  <xacro:property name="body_mass" value="25.0"/>
+  <xacro:property name="steer_servo_mass" value="0.3"/>
+  <!-- Arm parameters (5-DOF) -->
+  <xacro:property name="arm_base_height" value="0.20"/>
+  <xacro:property name="arm_link1_len" value="0.10"/>
+  <xacro:property name="arm_link2_len" value="0.18"/>
+  <xacro:property name="arm_link3_len" value="0.16"/>
+  <xacro:property name="arm_link4_len" value="0.12"/>
+  <xacro:property name="arm_link5_len" value="0.08"/>
+  <xacro:property name="arm_joint_limits" value="{'j1':3.14,'j2':1.6,'j3':1.6,'j4':3.14,'j5':3.14}"/>
+  <!-- Misc -->
+  <xacro:property name="encoder_cpr" value="1024"/>  <!-- counts per rev -->
+  <xacro:property name="wheel_inertia" value="0.02"/>
+  <xacro:property name="frame_prefix" value=""/>     <!-- set if you want a prefix for joint/link names -->
+  <!-- Helper macro: simple inertia for a box -->
+  <xacro:macro name="box_inertial" params="m lx ly lz">
     <inertial>
-      <mass value="25.0"/>
+      <mass value="${m}"/>
       <origin xyz="0 0 0"/>
-      <inertia ixx="1.0" ixy="0.0" ixz="0.0" iyy="1.0" iyz="0.0" izz="1.0"/>
+      <inertia ixx="${m*(ly*ly + lz*lz)/12.0}" ixy="0.0" ixz="0.0"
+               iyy="${m*(lx*lx + lz*lz)/12.0}" iyz="0.0"
+               izz="${m*(lx*lx + ly*ly)/12.0}"/>
     </inertial>
-  </link>
-  <!-- Front-left steering -->
-  <link name="fl_steer_link"/>
-  <joint name="fl_steer_joint" type="continuous">
-    <parent link="base_link"/>
-    <child link="fl_steer_link"/>
-    <origin xyz="0.35 0.25 0.0" rpy="0 0 0"/>
+  </xacro:macro>
+  <!-- ========= base link ========= -->
+  <link name="${frame_prefix}base_link">
+    <visual>
+      <origin xyz="0 0 ${base_height/2.0}" rpy="0 0 0"/>
+      <geometry>
+        <box size="${base_length} ${base_width} ${base_height}"/>
+      </geometry>
+      <material name="blue"/>
+    </visual>
+    <collision>
+      <origin xyz="0 0 ${base_height/2.0}" rpy="0 0 0"/>
+      <geometry>
+        <box size="${base_length} ${base_width} ${base_height}"/>
+      </geometry>
+    </collision>
+    <!-- inertial -->
+    <xacro:box_inertial m="${body_mass}" lx="${base_length}" ly="${base_width}" lz="${base_height}"/>
+  </link>
+  <!-- ========= helper: wheel model ========= -->
+  <xacro:macro name="wheel" params="side name x y">
+    <link name="${frame_prefix}${name}_wheel_link">
+      <visual>
+        <origin xyz="0 0 0" rpy="0 0 0"/>
+        <geometry>
+          <cylinder length="${wheel_thickness}" radius="${wheel_radius}"/>
+        </geometry>
+      </visual>
+      <collision>
+        <origin xyz="0 0 0" rpy="0 0 0"/>
+        <geometry>
+          <cylinder length="${wheel_thickness}" radius="${wheel_radius}"/>
+        </geometry>
+      </collision>
+      <inertial>
+        <mass value="${wheel_mass}"/>
+        <origin xyz="0 0 0"/>
+        <inertia ixx="${wheel_inertia}" ixy="0" ixz="0" iyy="${wheel_inertia}" iyz="0" izz="${wheel_inertia}"/>
+      </inertial>
+    </link>
+    <!-- wheel revolute joint (rotation axis Y for rolling) -->
+    <joint name="${frame_prefix}${name}_wheel_joint" type="continuous">
+      <parent link="${frame_prefix}${side}_steer_link"/>
+      <child link="${frame_prefix}${name}_wheel_link"/>
+      <!-- wheel is located at x,y relative to steer link's origin -->
+      <origin xyz="${x} ${y} 0" rpy="0 0 0"/>
+      <axis xyz="0 1 0"/>
+    </joint>
+  </xacro:macro>
+  <!-- ========= helper: steer block ========= -->
+  <xacro:macro name="steer_block" params="side steer_name steer_joint_x steer_joint_y">
+    <link name="${frame_prefix}${side}_steer_link">
+      <visual>
+        <origin xyz="0 0 0" rpy="0 0 0"/>
+        <geometry>
+          <box size="0.06 0.08 0.06"/>
+        </geometry>
+      </visual>
+      <collision>
+        <origin xyz="0 0 0" rpy="0 0 0"/>
+        <geometry>
+          <box size="0.06 0.08 0.06"/>
+        </geometry>
+      </collision>
+      <inertial>
+        <mass value="${steer_servo_mass}"/>
+        <origin xyz="0 0 0"/>
+        <inertia ixx="0.001" ixy="0.0" ixz="0.0" iyy="0.001" iyz="0.0" izz="0.001"/>
+      </inertial>
+    </link>
+    <joint name="${frame_prefix}${side}_steer_joint" type="continuous">
+      <parent link="${frame_prefix}base_link"/>
+      <child link="${frame_prefix}${side}_steer_link"/>
+      <origin xyz="${steer_joint_x} ${steer_joint_y} 0" rpy="0 0 0"/>
+      <axis xyz="0 0 1"/>
+    </joint>
+  </xacro:macro>
+  <!-- ========= instantiate steer blocks and wheels ========= -->
+  <!-- Left front -->
+  <xacro:steer_block side="fl" steer_name="fl_steer" steer_joint_x="${front_axle_x}" steer_joint_y="${half_track}"/>
+  <xacro:wheel side="fl" name="fl" x="0 0 0" y="0"/>
+  <!-- Left middle (no steer, attach directly to base_link) -->
+  <link name="${frame_prefix}ml_steer_link">
+    <visual>
+      <origin xyz="0 0 0" rpy="0 0 0"/>
+      <geometry>
+        <box size="0.02 0.02 0.02"/>
+      </geometry>
+    </visual>
+    <inertial>
+      <mass value="0.05"/>
+      <origin xyz="0 0 0"/>
+      <inertia ixx="1e-4" ixy="0" ixz="0" iyy="1e-4" iyz="0" izz="1e-4"/>
+    </inertial>
+  </link>
+  <joint name="${frame_prefix}ml_mount_joint" type="fixed">
+    <parent link="${frame_prefix}base_link"/>
+    <child link="${frame_prefix}ml_steer_link"/>
+    <origin xyz="${mid_axle_x} ${half_track} 0" rpy="0 0 0"/>
+  </joint>
+  <xacro:wheel side="ml" name="ml" x="0 0 0" y="0"/>
+  <!-- Left rear -->
+  <xacro:steer_block side="rl" steer_name="rl_steer" steer_joint_x="${rear_axle_x}" steer_joint_y="${half_track}"/>
+  <xacro:wheel side="rl" name="rl" x="0 0 0" y="0"/>
+  <!-- Right side: mirror y coordinate to -half_track -->
+  <xacro:steer_block side="fr" steer_name="fr_steer" steer_joint_x="${front_axle_x}" steer_joint_y="${-half_track}"/>
+  <xacro:wheel side="fr" name="fr" x="0 0 0" y="0"/>
+  <link name="${frame_prefix}mr_steer_link">
+    <visual>
+      <origin xyz="0 0 0" rpy="0 0 0"/>
+      <geometry>
+        <box size="0.02 0.02 0.02"/>
+      </geometry>
+    </visual>
+    <inertial>
+      <mass value="0.05"/>
+      <origin xyz="0 0 0"/>
+      <inertia ixx="1e-4" ixy="0" ixz="0" iyy="1e-4" iyz="0" izz="1e-4"/>
+    </inertial>
+  </link>
+  <joint name="${frame_prefix}mr_mount_joint" type="fixed">
+    <parent link="${frame_prefix}base_link"/>
+    <child link="${frame_prefix}mr_steer_link"/>
+    <origin xyz="${mid_axle_x} ${-half_track} 0" rpy="0 0 0"/>
+  </joint>
+  <xacro:wheel side="mr" name="mr" x="0 0 0" y="0"/>
+  <xacro:steer_block side="rr" steer_name="rr_steer" steer_joint_x="${rear_axle_x}" steer_joint_y="${-half_track}"/>
+  <xacro:wheel side="rr" name="rr" x="0 0 0" y="0"/>
+  <!-- Note: wheel macros created wheel links named <name>_wheel_link and joints named <name>_wheel_joint.
+       For the middle wheels, we used ml and mr similarly but attached to ml_steer_link and mr_steer_link respectively.
+  -->
+  <!-- ========= Transmissions for ros_control (velocity for wheel joints, position for steering) ========= -->
+  <!-- Wheel velocity transmissions (6 wheels) -->
+  <transmission name="${frame_prefix}fl_wheel_trans">
+    <type>transmission_interface/SimpleTransmission</type>
+    <joint name="${frame_prefix}fl_wheel_joint"/>
+    <actuator name="${frame_prefix}fl_wheel_motor">
+      <mechanicalReduction>1</mechanicalReduction>
+    </actuator>
+  </transmission>
+  <transmission name="${frame_prefix}ml_wheel_trans">
+    <type>transmission_interface/SimpleTransmission</type>
+    <joint name="${frame_prefix}ml_wheel_joint"/>
+    <actuator name="${frame_prefix}ml_wheel_motor"><mechanicalReduction>1</mechanicalReduction></actuator>
+  </transmission>
+  <transmission name="${frame_prefix}rl_wheel_trans">
+    <type>transmission_interface/SimpleTransmission</type>
+    <joint name="${frame_prefix}rl_wheel_joint"/>
+    <actuator name="${frame_prefix}rl_wheel_motor"><mechanicalReduction>1</mechanicalReduction></actuator>
+  </transmission>
+  <transmission name="${frame_prefix}fr_wheel_trans">
+    <type>transmission_interface/SimpleTransmission</type>
+    <joint name="${frame_prefix}fr_wheel_joint"/>
+    <actuator name="${frame_prefix}fr_wheel_motor"><mechanicalReduction>1</mechanicalReduction></actuator>
+  </transmission>
+  <transmission name="${frame_prefix}mr_wheel_trans">
+    <type>transmission_interface/SimpleTransmission</type>
+    <joint name="${frame_prefix}mr_wheel_joint"/>
+    <actuator name="${frame_prefix}mr_wheel_motor"><mechanicalReduction>1</mechanicalReduction></actuator>
+  </transmission>
+  <transmission name="${frame_prefix}rr_wheel_trans">
+    <type>transmission_interface/SimpleTransmission</type>
+    <joint name="${frame_prefix}rr_wheel_joint"/>
+    <actuator name="${frame_prefix}rr_wheel_motor"><mechanicalReduction>1</mechanicalReduction></actuator>
+  </transmission>
+  <!-- Steering transmissions (position control) -->
+  <transmission name="${frame_prefix}fl_steer_trans">
+    <type>transmission_interface/SimpleTransmission</type>
+    <joint name="${frame_prefix}fl_steer_joint"/>
+    <actuator name="${frame_prefix}fl_steer_servo"/>
+  </transmission>
+  <transmission name="${frame_prefix}fr_steer_trans">
+    <type>transmission_interface/SimpleTransmission</type>
+    <joint name="${frame_prefix}fr_steer_joint"/>
+    <actuator name="${frame_prefix}fr_steer_servo"/>
+  </transmission>
+  <transmission name="${frame_prefix}rl_steer_trans">
+    <type>transmission_interface/SimpleTransmission</type>
+    <joint name="${frame_prefix}rl_steer_joint"/>
+    <actuator name="${frame_prefix}rl_steer_servo"/>
+  </transmission>
+  <transmission name="${frame_prefix}rr_steer_trans">
+    <type>transmission_interface/SimpleTransmission</type>
+    <joint name="${frame_prefix}rr_steer_joint"/>
+    <actuator name="${frame_prefix}rr_steer_servo"/>
+  </transmission>
+  <!-- ========= 5-DOF ARM (front center) ========= -->
+  <link name="${frame_prefix}arm_base_link">
+    <visual>
+      <origin xyz="0 0 0" rpy="0 0 0"/>
+      <geometry>
+        <cylinder radius="0.05" length="0.04"/>
+      </geometry>
+    </visual>
+    <collision>
+      <origin xyz="0 0 0" rpy="0 0 0"/>
+      <geometry>
+        <cylinder radius="0.05" length="0.04"/>
+      </geometry>
+    </collision>
+    <inertial>
+      <mass value="1.2"/>
+      <origin xyz="0 0 0"/>
+      <inertia ixx="0.02" ixy="0" ixz="0" iyy="0.02" iyz="0" izz="0.02"/>
+    </inertial>
+  </link>
+  <joint name="${frame_prefix}arm_base_fixed" type="fixed">
+    <parent link="${frame_prefix}base_link"/>
+    <child link="${frame_prefix}arm_base_link"/>
+    <origin xyz="${front_axle_x + 0.1} 0 ${arm_base_height}" rpy="0 0 0"/>
+  </joint>
+  <!-- arm joint 1: rotate about Z (base yaw) -->
+  <link name="${frame_prefix}arm_link_1"/>
+  <joint name="${frame_prefix}arm_joint_1" type="revolute">
+    <parent link="${frame_prefix}arm_base_link"/>
+    <child link="${frame_prefix}arm_link_1"/>
+    <origin xyz="0 0 0.02" rpy="0 0 0"/>
     <axis xyz="0 0 1"/>
-  </joint>
-  <!-- Front-left wheel -->
-  <link name="fl_wheel_link"/>
-  <joint name="fl_wheel_joint" type="continuous">
-    <parent link="fl_steer_link"/>
-    <child link="fl_wheel_link"/>
-    <origin xyz="0 0 -0.08" rpy="0 0 0"/>
+    <limit lower="-3.1416" upper="3.1416" effort="50" velocity="1.0"/>
+  </joint>
+  <!-- arm link visuals + inertials (simple cylinders) -->
+  <link name="${frame_prefix}arm_link_2">
+    <visual>
+      <origin xyz="${arm_link1_len/2.0} 0 0" rpy="0 0 0"/>
+      <geometry><cylinder radius="0.03" length="${arm_link1_len}"/></geometry>
+    </visual>
+    <inertial><mass value="0.6"/><origin xyz="${arm_link1_len/2.0} 0 0"/><inertia ixx="0.001" ixy="0" ixz="0" iyy="0.001" iyz="0" izz="0.001"/></inertial>
+  </link>
+  <joint name="${frame_prefix}arm_joint_2" type="revolute">
+    <parent link="${frame_prefix}arm_link_1"/>
+    <child link="${frame_prefix}arm_link_2"/>
+    <origin xyz="0 0 0" rpy="0 0 0"/>
     <axis xyz="0 1 0"/>
-  </joint>
-  <!-- Arm base (front center) -->
-  <link name="arm_base_link"/>
-  <joint name="arm_base_joint" type="fixed">
-    <parent link="base_link"/>
-    <child link="arm_base_link"/>
-    <origin xyz="0.45 0 0.2"/>
-  </joint>
-  <!-- Add rest of wheels, steers and arm joints similarly -->
+    <limit lower="-1.57" upper="1.57" effort="30" velocity="1.0"/>
+  </joint>
+  <link name="${frame_prefix}arm_link_3">
+    <visual>
+      <origin xyz="${arm_link2_len/2.0} 0 0" rpy="0 0 0"/>
+      <geometry><cylinder radius="0.03" length="${arm_link2_len}"/></geometry>
+    </visual>
+    <inertial><mass value="0.5"/><origin xyz="${arm_link2_len/2.0} 0 0"/></inertial>
+  </link>
+  <joint name="${frame_prefix}arm_joint_3" type="revolute">
+    <parent link="${frame_prefix}arm_link_2"/>
+    <child link="${frame_prefix}arm_link_3"/>
+    <origin xyz="${arm_link1_len} 0 0" rpy="0 0 0"/>
+    <axis xyz="0 1 0"/>
+    <limit lower="-1.57" upper="1.57" effort="20" velocity="1.0"/>
+  </joint>
+  <link name="${frame_prefix}arm_link_4">
+    <visual>
+      <origin xyz="${arm_link3_len/2.0} 0 0" rpy="0 0 0"/>
+      <geometry><cylinder radius="0.025" length="${arm_link3_len}"/></geometry>
+    </visual>
+    <inertial><mass value="0.3"/><origin xyz="${arm_link3_len/2.0} 0 0"/></inertial>
+  </link>
+  <joint name="${frame_prefix}arm_joint_4" type="revolute">
+    <parent link="${frame_prefix}arm_link_3"/>
+    <child link="${frame_prefix}arm_link_4"/>
+    <origin xyz="${arm_link2_len} 0 0" rpy="0 0 0"/>
+    <axis xyz="0 1 0"/>
+    <limit lower="-3.14" upper="3.14" effort="10" velocity="2.0"/>
+  </joint>
+  <link name="${frame_prefix}arm_link_5">
+    <visual>
+      <origin xyz="${arm_link4_len/2.0} 0 0" rpy="0 0 0"/>
+      <geometry><cylinder radius="0.02" length="${arm_link4_len}"/></geometry>
+    </visual>
+    <inertial><mass value="0.15"/><origin xyz="${arm_link4_len/2.0} 0 0"/></inertial>
+  </link>
+  <joint name="${frame_prefix}arm_joint_5" type="revolute">
+    <parent link="${frame_prefix}arm_link_4"/>
+    <child link="${frame_prefix}arm_link_5"/>
+    <origin xyz="${arm_link3_len} 0 0" rpy="0 0 0"/>
+    <axis xyz="1 0 0"/>
+    <limit lower="-3.14" upper="3.14" effort="5" velocity="3.0"/>
+  </joint>
+  <link name="${frame_prefix}arm_ee_link">
+    <visual><origin xyz="${arm_link4_len} 0 0" rpy="0 0 0"><geometry><sphere radius="0.03"/></geometry></origin></visual>
+  </link>
+  <joint name="${frame_prefix}arm_ee_fixed" type="fixed">
+    <parent link="${frame_prefix}arm_link_5"/>
+    <child link="${frame_prefix}arm_ee_link"/>
+    <origin xyz="${arm_link5_len} 0 0" rpy="0 0 0"/>
+  </joint>
+  <!-- Arm transmissions (create one transmission per arm joint) -->
+  <transmission name="${frame_prefix}arm_joint_1_trans">
+    <type>transmission_interface/SimpleTransmission</type>
+    <joint name="${frame_prefix}arm_joint_1"/>
+    <actuator name="${frame_prefix}arm_joint_1_motor"/>
+  </transmission>
+  <transmission name="${frame_prefix}arm_joint_2_trans">
+    <type>transmission_interface/SimpleTransmission</type>
+    <joint name="${frame_prefix}arm_joint_2"/>
+    <actuator name="${frame_prefix}arm_joint_2_motor"/>
+  </transmission>
+  <transmission name="${frame_prefix}arm_joint_3_trans">
+    <type>transmission_interface/SimpleTransmission</type>
+    <joint name="${frame_prefix}arm_joint_3"/>
+    <actuator name="${frame_prefix}arm_joint_3_motor"/>
+  </transmission>
+  <transmission name="${frame_prefix}arm_joint_4_trans">
+    <type>transmission_interface/SimpleTransmission</type>
+    <joint name="${frame_prefix}arm_joint_4"/>
+    <actuator name="${frame_prefix}arm_joint_4_motor"/>
+  </transmission>
+  <transmission name="${frame_prefix}arm_joint_5_trans">
+    <type>transmission_interface/SimpleTransmission</type>
+    <joint name="${frame_prefix}arm_joint_5"/>
+    <actuator name="${frame_prefix}arm_joint_5_motor"/>
+  </transmission>
+  <!-- ========= Sensors (URDF links & Gazebo plugin stubs) ========= -->
+  <!-- IMU link (attached to base) -->
+  <link name="${frame_prefix}imu_link">
+    <visual><origin xyz="0 0 0.06"/><geometry><box size="0.02 0.02 0.01"/></geometry></visual>
+    <inertial><mass value="0.02"/><origin xyz="0 0 0.06"/></inertial>
+  </link>
+  <joint name="${frame_prefix}imu_joint" type="fixed">
+    <parent link="${frame_prefix}base_link"/>
+    <child link="${frame_prefix}imu_link"/>
+    <origin xyz="0 0 0.06" rpy="0 0 0"/>
+  </joint>
+  <!-- Kinect RGB-D camera -->
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